File: PCB/3k/KiCad Files/project.kicad_sch (KiCad schematic)
At the start: 39 parts, among them K1 Hall_Sensor, K2 Hall_Sensor, K3 Hall_Sensor, SW1 BOOTSEL, SW2 RESET, U1 RP2040, U2 SRV05-4, U3 XC6206PxxxMR, U4 W25Q128JVS, Y1 12MHZ

Commit message: Add libraries
Other:
- note added: "Box for RGBs Coming soon."
- note added: "Crystal"
- note added: "Decoupling Caps"
- note added: "ESD"
- note added: "Flash Memory"
- note added: "Hall Sensors"
- note added: "Mounting Hole for switches"
- note added: "RESET"
- note added: "RP2040"
- note added: "USB-C"
- note added: "Voltage Regulator"
- moved on the sheet: H1, H2, H3
